File: kicad/adc/adc.sch (KiCad schematic (older format))
At the start: 5 parts, among them J1 +5V Isense, J2 +3.3V Isense, J3 DE10 Nano GPIO 0/1

Commit message: PCB routed
Parts:
- J3: footprint (none) -> Connector_PinSocket_2.54mm:PinSocket_2x20_P2.54mm_Vertical
Connections:
- net labels added: ADC1-CLK, ADC1-D0, ADC1-D1, ADC1-D2, ADC1-D3, ADC1-D4, ADC1-D5, ADC1-D6, ADC1-D7, ADC2-CLK, ADC2-D0, ADC2-D1, ADC2-D2, ADC2-D3, ADC2-D4, ADC2-D5, ADC2-D6, ADC2-D7, ADC3-CLK, ADC3-D0, ADC3-D1, ADC3-D2, ADC3-D3, ADC3-D4, ADC3-D5, ADC3-D6, ADC3-D7, ADC4-CLK, ADC4-D0, ADC4-D1, ADC4-D2, ADC4-D3, ADC4-D4, ADC4-D5, ADC4-D6, ADC4-D7
- wire segments 128 -> 92
