File: kicad/adc/adc1.sch (KiCad schematic (older format))
At the start: 55 parts, among them J4 analog in, J5 disable jumper, U1 ADA4891, U2 MIC5219-adj, U3 ADC1175-50

Commit message: fixed OpAmp power supply and added another decoupling capacitor
Parts:
- added C2: 100n, Capacitor_SMD:C_0805_2012Metric, symbol Device:C
- C6: renamed from C5; value 470p -> 47p
- renumbered C9 to C10, C10 to C11, C11 to C12, C12 to C13, C13 to C14, C14 to C15, C2 to C3, C3 to C4, C4 to C5, C6 to C7, C7 to C8, C8 to C9
Connections:
- wire segments 152 -> 153

Commit message: PCB routed
Parts:
- C1: footprint Capacitor_SMD:C_0805_2012Metric -> Capacitor_SMD:C_1206_3216Metric
- C10, C11, C14, C5, C8, C9: footprint Capacitor_SMD:C_1206_3216Metric -> Capacitor_SMD:C_0805_2012Metric
- D1, D2: footprint Diode_THT:D_DO-201AE_P15.24mm_Horizontal -> Diode_SMD:D_SMA_Handsoldering
- F1: footprint (none) -> Fuse:Fuse_2512_6332Metric
- RV1, RV2: footprint (none) -> Potentiometer_SMD:Potentiometer_Bourns_3269P_Horizontal
- TP1, TP10, TP2, TP3, TP4, TP5, TP6, TP7, TP8, TP9: footprint (none) -> TestPoint:TestPoint_Pad_2.0x2.0mm
Connections:
- net labels removed: 4V
- wire segments 153 -> 157
Other:
- note added: "4 V"

Commit message: first working FPGA version with Python test script
Parts:
- C3: value 2p, TBD -> 0.5p
- R10, R11, R5: value 0 -> n.p.
- R4: value 20 -> 33
