File: kicad/adc/adc.kicad_pcb (KiCad board)
At the start: 2 copper layers, 49 parts, among them J1 conn, J2 analog in, U1 ADA4622-1, U2 LMH6702, U3 LMH6702, U4 ADC1175

Commit message: PCB routed
Parts:
- added C20: 10u, Capacitor_SMD:C_0805_2012Metric, F.Cu at (196.2, 89.2)
- added C21: 47p, Capacitor_SMD:C_0805_2012Metric, F.Cu at (208.9, 88.3)
- added C22: 470p, Capacitor_SMD:C_0805_2012Metric, F.Cu at (212.1, 79.4)
- added C23: 1u, Capacitor_SMD:C_0805_2012Metric, F.Cu at (210.8, 83.2)
- added C24: 1u, Capacitor_SMD:C_0805_2012Metric, F.Cu at (216.5, 91.4)
- added C25: 1u, Capacitor_SMD:C_0805_2012Metric, F.Cu at (215.9, 75.9)
- added C26: 10u, Capacitor_SMD:C_0805_2012Metric, F.Cu at (220.6, 80.6)
- added C27: 100n, Capacitor_SMD:C_0805_2012Metric, F.Cu at (220.6, 83.2)
- added C28: 100n, Capacitor_SMD:C_0805_2012Metric, F.Cu at (233.0, 79.7)
- added C29: 10u, Capacitor_SMD:C_0805_2012Metric, F.Cu at (230.5, 80.3)
- added C30: 100n, Capacitor_SMD:C_0805_2012Metric, F.Cu at (228.0, 80.3)
- added C31: n.p., Capacitor_SMD:C_1206_3216Metric, F.Cu at (192.7, 106.0)
- added C32: 100n, Capacitor_SMD:C_0805_2012Metric, F.Cu at (211.1, 95.9)
- added C33: 2p, TBD, Capacitor_SMD:C_0805_2012Metric, F.Cu at (199.4, 105.4)
- added C34: 100n, Capacitor_SMD:C_0805_2012Metric, F.Cu at (201.0, 112.4)
- added C35: 10u, Capacitor_SMD:C_0805_2012Metric, F.Cu at (196.2, 113.3)
- added C36: 47p, Capacitor_SMD:C_0805_2012Metric, F.Cu at (208.9, 112.4)
- added C37: 470p, Capacitor_SMD:C_0805_2012Metric, F.Cu at (212.1, 103.5)
- added C38: 1u, Capacitor_SMD:C_0805_2012Metric, F.Cu at (210.8, 107.3)
- added C39: 1u, Capacitor_SMD:C_0805_2012Metric, F.Cu at (216.5, 115.6)
- added C40: 1u, Capacitor_SMD:C_0805_2012Metric, F.Cu at (215.9, 100.0)
- added C41: 10u, Capacitor_SMD:C_0805_2012Metric, F.Cu at (220.6, 104.8)
- added C42: 100n, Capacitor_SMD:C_0805_2012Metric, F.Cu at (220.6, 107.3)
- added C43: 100n, Capacitor_SMD:C_0805_2012Metric, F.Cu at (233.0, 103.8)
- added C44: 10u, Capacitor_SMD:C_0805_2012Metric, F.Cu at (230.5, 104.4)
- added C45: 100n, Capacitor_SMD:C_0805_2012Metric, F.Cu at (228.0, 104.4)
- added C46: n.p., Capacitor_SMD:C_1206_3216Metric, F.Cu at (192.7, 130.2)
- added C47: 100n, Capacitor_SMD:C_0805_2012Metric, F.Cu at (211.1, 120.0)
- added C48: 2p, TBD, Capacitor_SMD:C_0805_2012Metric, F.Cu at (199.4, 129.5)
- added C49: 100n, Capacitor_SMD:C_0805_2012Metric, F.Cu at (201.0, 136.5)
- added C50: 10u, Capacitor_SMD:C_0805_2012Metric, F.Cu at (196.2, 137.5)
- added C51: 47p, Capacitor_SMD:C_0805_2012Metric, F.Cu at (208.9, 136.5)
- added C52: 470p, Capacitor_SMD:C_0805_2012Metric, F.Cu at (212.1, 127.6)
- added C53: 1u, Capacitor_SMD:C_0805_2012Metric, F.Cu at (210.8, 131.5)
- added C54: 1u, Capacitor_SMD:C_0805_2012Metric, F.Cu at (216.5, 139.7)
- added C55: 1u, Capacitor_SMD:C_0805_2012Metric, F.Cu at (215.9, 124.1)
- added C56: 10u, Capacitor_SMD:C_0805_2012Metric, F.Cu at (220.6, 128.9)
- added C57: 100n, Capacitor_SMD:C_0805_2012Metric, F.Cu at (220.6, 131.5)
- added C58: 100n, Capacitor_SMD:C_0805_2012Metric, F.Cu at (233.0, 127.9)
- added C59: 10u, Capacitor_SMD:C_0805_2012Metric, F.Cu at (230.5, 128.6)
- added C60: 100n, Capacitor_SMD:C_0805_2012Metric, F.Cu at (228.0, 128.6)
- added D2: SM4T15AY, Diode_SMD:D_SMA_Handsoldering, F.Cu at (186.7, 50.8)
- added D3: SM4T15AY, Diode_SMD:D_SMA_Handsoldering, F.Cu at (187.3, 85.1)
- added D4: SM4T15AY, Diode_SMD:D_SMA_Handsoldering, F.Cu at (186.7, 74.9)
- added D5: SM4T15AY, Diode_SMD:D_SMA_Handsoldering, F.Cu at (187.3, 109.2)
- added D6: SM4T15AY, Diode_SMD:D_SMA_Handsoldering, F.Cu at (186.7, 99.1)
- added D7: SM4T15AY, Diode_SMD:D_SMA_Handsoldering, F.Cu at (187.3, 133.4)
- added D8: SM4T15AY, Diode_SMD:D_SMA_Handsoldering, F.Cu at (186.7, 123.2)
- added F1: Fuse, Fuse:Fuse_2512_6332Metric, F.Cu at (181.6, 61.0)
- added F2: Fuse, Fuse:Fuse_2512_6332Metric, F.Cu at (181.6, 85.1)
- added F3: Fuse, Fuse:Fuse_2512_6332Metric, F.Cu at (181.6, 109.2)
- added F4: Fuse, Fuse:Fuse_2512_6332Metric, F.Cu at (181.6, 133.4)
- added J10: analog in, Connector_PinHeader_2.54mm:PinHeader_1x02_P2.54mm_Vertical, F.Cu at (181.6, 121.9)
- added J11: disable jumper, Connector_PinHeader_2.54mm:PinHeader_1x02_P2.54mm_Vertical, F.Cu at (238.8, 120.0)
- added J3: DE10 Nano GPIO 0/1, Connector_PinSocket_2.54mm:PinSocket_2x20_P2.54mm_Vertical, B.Cu at (265.4, 116.8)
- added J4: analog in, Connector_PinHeader_2.54mm:PinHeader_1x02_P2.54mm_Vertical, F.Cu at (181.6, 49.5)
- added J5: disable jumper, Connector_PinHeader_2.54mm:PinHeader_1x02_P2.54mm_Vertical, F.Cu at (238.8, 47.6)
- added J6: analog in, Connector_PinHeader_2.54mm:PinHeader_1x02_P2.54mm_Vertical, F.Cu at (181.6, 73.7)
- added J7: disable jumper, Connector_PinHeader_2.54mm:PinHeader_1x02_P2.54mm_Vertical, F.Cu at (238.8, 71.8)
- added J8: analog in, Connector_PinHeader_2.54mm:PinHeader_1x02_P2.54mm_Vertical, F.Cu at (181.6, 97.8)
- added J9: disable jumper, Connector_PinHeader_2.54mm:PinHeader_1x02_P2.54mm_Vertical, F.Cu at (238.8, 95.9)
- added L3: BLM31KN801SN1L, Inductor_SMD:L_1206_3216Metric, F.Cu at (226.7, 74.4)
- added L4: BLM31KN801SN1L, Inductor_SMD:L_1206_3216Metric, F.Cu at (225.4, 79.7)
- added L5: BLM31KN801SN1L, Inductor_SMD:L_1206_3216Metric, F.Cu at (226.7, 98.6)
- added L6: BLM31KN801SN1L, Inductor_SMD:L_1206_3216Metric, F.Cu at (225.4, 103.8)
- added L7: BLM31KN801SN1L, Inductor_SMD:L_1206_3216Metric, F.Cu at (226.7, 122.7)
- added L8: BLM31KN801SN1L, Inductor_SMD:L_1206_3216Metric, F.Cu at (225.4, 128.0)
- added R20: 33, Resistor_SMD:R_0805_2012Metric, F.Cu at (240.7, 59.1)
- added R21: 33, Resistor_SMD:R_0805_2012Metric, F.Cu at (236.9, 57.8)
- added R22: 150k, Resistor_SMD:R_1206_3216Metric, F.Cu at (192.9, 85.1)
- added R23: 20, Resistor_SMD:R_0805_2012Metric, F.Cu at (205.4, 87.6)
- added R24: 0, Resistor_SMD:R_0805_2012Metric, F.Cu at (204.5, 83.2)
- added R25: 0, Resistor_SMD:R_0805_2012Metric, F.Cu at (207.6, 83.2)
- added R26: 4k5, Resistor_SMD:R_0805_2012Metric, F.Cu at (218.4, 75.9)
- added R27: 10k, Resistor_SMD:R_0805_2012Metric, F.Cu at (221.0, 75.9)
- added R28: 0, Resistor_SMD:R_0805_2012Metric, F.Cu at (220.6, 91.4)
- added R29: 0, Resistor_SMD:R_0805_2012Metric, F.Cu at (216.5, 84.5)
- added R30: 0, Resistor_SMD:R_0805_2012Metric, F.Cu at (220.6, 88.9)
- added R31: 10k, Resistor_SMD:R_0805_2012Metric, F.Cu at (230.8, 76.2)
- added R32: 33, Resistor_SMD:R_0805_2012Metric, F.Cu at (236.9, 92.1)
- added R33: 33, Resistor_SMD:R_0805_2012Metric, F.Cu at (240.7, 90.8)
- added R34: 33, Resistor_SMD:R_0805_2012Metric, F.Cu at (236.9, 89.5)
- added R35: 33, Resistor_SMD:R_0805_2012Metric, F.Cu at (240.7, 88.3)
- added R36: 33, Resistor_SMD:R_0805_2012Metric, F.Cu at (236.9, 87.0)
- added R37: 33, Resistor_SMD:R_0805_2012Metric, F.Cu at (240.7, 85.7)
- added R38: 33, Resistor_SMD:R_0805_2012Metric, F.Cu at (236.9, 84.5)
- added R39: 33, Resistor_SMD:R_0805_2012Metric, F.Cu at (240.7, 83.2)
- added R40: 33, Resistor_SMD:R_0805_2012Metric, F.Cu at (236.9, 81.9)
- added R41: 150k, Resistor_SMD:R_1206_3216Metric, F.Cu at (192.9, 109.2)
- added R42: 20, Resistor_SMD:R_0805_2012Metric, F.Cu at (205.4, 111.8)
- added R43: 0, Resistor_SMD:R_0805_2012Metric, F.Cu at (204.5, 107.3)
- added R44: 0, Resistor_SMD:R_0805_2012Metric, F.Cu at (207.6, 107.3)
- added R45: 4k5, Resistor_SMD:R_0805_2012Metric, F.Cu at (218.4, 100.0)
- added R46: 10k, Resistor_SMD:R_0805_2012Metric, F.Cu at (221.0, 100.0)
- added R47: 0, Resistor_SMD:R_0805_2012Metric, F.Cu at (220.6, 115.6)
- added R48: 0, Resistor_SMD:R_0805_2012Metric, F.Cu at (216.5, 108.6)
- added R49: 0, Resistor_SMD:R_0805_2012Metric, F.Cu at (220.6, 113.0)
- added R50: 10k, Resistor_SMD:R_0805_2012Metric, F.Cu at (230.8, 100.3)
- added R51: 33, Resistor_SMD:R_0805_2012Metric, F.Cu at (236.9, 116.2)
- added R52: 33, Resistor_SMD:R_0805_2012Metric, F.Cu at (240.7, 114.9)
- added R53: 33, Resistor_SMD:R_0805_2012Metric, F.Cu at (236.9, 113.7)
- added R54: 33, Resistor_SMD:R_0805_2012Metric, F.Cu at (240.7, 112.4)
- added R55: 33, Resistor_SMD:R_0805_2012Metric, F.Cu at (236.9, 111.1)
- added R56: 33, Resistor_SMD:R_0805_2012Metric, F.Cu at (240.7, 109.9)
- added R57: 33, Resistor_SMD:R_0805_2012Metric, F.Cu at (236.9, 108.6)
- added R58: 33, Resistor_SMD:R_0805_2012Metric, F.Cu at (240.7, 107.3)
- added R59: 33, Resistor_SMD:R_0805_2012Metric, F.Cu at (236.9, 106.0)
- added R60: 150k, Resistor_SMD:R_1206_3216Metric, F.Cu at (192.9, 133.4)
- added R61: 20, Resistor_SMD:R_0805_2012Metric, F.Cu at (205.4, 135.9)
- added R62: 0, Resistor_SMD:R_0805_2012Metric, F.Cu at (204.5, 131.5)
- added R63: 0, Resistor_SMD:R_0805_2012Metric, F.Cu at (207.6, 131.5)
- added R64: 4k5, Resistor_SMD:R_0805_2012Metric, F.Cu at (218.4, 124.2)
- added R65: 10k, Resistor_SMD:R_0805_2012Metric, F.Cu at (221.0, 124.1)
- added R66: 0, Resistor_SMD:R_0805_2012Metric, F.Cu at (220.6, 139.7)
- added R67: 0, Resistor_SMD:R_0805_2012Metric, F.Cu at (216.5, 132.7)
- added R68: 0, Resistor_SMD:R_0805_2012Metric, F.Cu at (220.6, 137.2)
- added R69: 10k, Resistor_SMD:R_0805_2012Metric, F.Cu at (230.8, 124.5)
- added R70: 33, Resistor_SMD:R_0805_2012Metric, F.Cu at (236.8, 140.3)
- added R71: 33, Resistor_SMD:R_0805_2012Metric, F.Cu at (240.7, 139.1)
- added R72: 33, Resistor_SMD:R_0805_2012Metric, F.Cu at (236.8, 137.8)
- added R73: 33, Resistor_SMD:R_0805_2012Metric, F.Cu at (240.7, 136.5)
- added R74: 33, Resistor_SMD:R_0805_2012Metric, F.Cu at (236.8, 135.3)
- added R75: 33, Resistor_SMD:R_0805_2012Metric, F.Cu at (240.7, 134.0)
- added R76: 33, Resistor_SMD:R_0805_2012Metric, F.Cu at (236.8, 132.7)
- added R77: 33, Resistor_SMD:R_0805_2012Metric, F.Cu at (240.7, 131.5)
- added R78: 33, Resistor_SMD:R_0805_2012Metric, F.Cu at (236.8, 130.2)
- added RV3: 50k, Potentiometer_SMD:Potentiometer_Bourns_3269P_Horizontal, F.Cu at (205.1, 74.3)
- added RV4: 50k, Potentiometer_SMD:Potentiometer_Bourns_3269P_Horizontal, F.Cu at (197.5, 74.3)
- added RV5: 50k, Potentiometer_SMD:Potentiometer_Bourns_3269P_Horizontal, F.Cu at (205.1, 98.4)
- added RV6: 50k, Potentiometer_SMD:Potentiometer_Bourns_3269P_Horizontal, F.Cu at (197.5, 98.5)
- added RV7: 50k, Potentiometer_SMD:Potentiometer_Bourns_3269P_Horizontal, F.Cu at (205.1, 122.5)
- added RV8: 50k, Potentiometer_SMD:Potentiometer_Bourns_3269P_Horizontal, F.Cu at (197.5, 122.5)
- added TP1: TestPoint, TestPoint:TestPoint_Pad_2.0x2.0mm, F.Cu at (191.8, 53.3)
- added TP10: TestPoint, TestPoint:TestPoint_Pad_2.0x2.0mm, F.Cu at (240.7, 53.3)
- added TP11: TestPoint, TestPoint:TestPoint_Pad_2.0x2.0mm, F.Cu at (191.8, 77.5)
- added TP12: TestPoint, TestPoint:TestPoint_Pad_2.0x2.0mm, F.Cu at (215.9, 71.8)
- added TP13: TestPoint, TestPoint:TestPoint_Pad_2.0x2.0mm, F.Cu at (215.9, 88.3)
- added TP14: TestPoint, TestPoint:TestPoint_Pad_2.0x2.0mm, F.Cu at (219.7, 71.8)
- added TP15: TestPoint, TestPoint:TestPoint_Pad_2.0x2.0mm, F.Cu at (216.5, 80.0)
- added TP16: TestPoint, TestPoint:TestPoint_Pad_2.0x2.0mm, F.Cu at (212.1, 88.3)
- added TP17: TestPoint, TestPoint:TestPoint_Pad_2.0x2.0mm, F.Cu at (229.9, 71.8)
- added TP18: TestPoint, TestPoint:TestPoint_Pad_2.0x2.0mm, F.Cu at (236.2, 77.5)
- added TP19: TestPoint, TestPoint:TestPoint_Pad_2.0x2.0mm, F.Cu at (223.5, 71.8)
- added TP2: TestPoint, TestPoint:TestPoint_Pad_2.0x2.0mm, F.Cu at (215.9, 47.6)
- added TP20: TestPoint, TestPoint:TestPoint_Pad_2.0x2.0mm, F.Cu at (240.7, 77.5)
- added TP21: TestPoint, TestPoint:TestPoint_Pad_2.0x2.0mm, F.Cu at (191.8, 101.6)
- added TP22: TestPoint, TestPoint:TestPoint_Pad_2.0x2.0mm, F.Cu at (215.9, 95.9)
- added TP23: TestPoint, TestPoint:TestPoint_Pad_2.0x2.0mm, F.Cu at (215.9, 112.4)
- added TP24: TestPoint, TestPoint:TestPoint_Pad_2.0x2.0mm, F.Cu at (219.7, 95.9)
- added TP25: TestPoint, TestPoint:TestPoint_Pad_2.0x2.0mm, F.Cu at (216.5, 104.1)
- added TP26: TestPoint, TestPoint:TestPoint_Pad_2.0x2.0mm, F.Cu at (212.1, 112.4)
- added TP27: TestPoint, TestPoint:TestPoint_Pad_2.0x2.0mm, F.Cu at (229.9, 95.9)
- added TP28: TestPoint, TestPoint:TestPoint_Pad_2.0x2.0mm, F.Cu at (236.2, 101.6)
- added TP29: TestPoint, TestPoint:TestPoint_Pad_2.0x2.0mm, F.Cu at (223.5, 95.9)
- added TP3: TestPoint, TestPoint:TestPoint_Pad_2.0x2.0mm, F.Cu at (215.9, 64.1)
- added TP30: TestPoint, TestPoint:TestPoint_Pad_2.0x2.0mm, F.Cu at (240.7, 101.6)
- added TP31: TestPoint, TestPoint:TestPoint_Pad_2.0x2.0mm, F.Cu at (191.8, 125.7)
- added TP32: TestPoint, TestPoint:TestPoint_Pad_2.0x2.0mm, F.Cu at (215.9, 120.0)
- added TP33: TestPoint, TestPoint:TestPoint_Pad_2.0x2.0mm, F.Cu at (215.9, 136.5)
- added TP34: TestPoint, TestPoint:TestPoint_Pad_2.0x2.0mm, F.Cu at (219.7, 120.0)
- added TP35: TestPoint, TestPoint:TestPoint_Pad_2.0x2.0mm, F.Cu at (216.5, 128.3)
- added TP36: TestPoint, TestPoint:TestPoint_Pad_2.0x2.0mm, F.Cu at (212.1, 136.5)
- added TP37: TestPoint, TestPoint:TestPoint_Pad_2.0x2.0mm, F.Cu at (229.9, 120.0)
- added TP38: TestPoint, TestPoint:TestPoint_Pad_2.0x2.0mm, F.Cu at (236.2, 125.7)
- added TP39: TestPoint, TestPoint:TestPoint_Pad_2.0x2.0mm, F.Cu at (223.5, 120.0)
- added TP4: TestPoint, TestPoint:TestPoint_Pad_2.0x2.0mm, F.Cu at (219.7, 47.6)
- added TP40: TestPoint, TestPoint:TestPoint_Pad_2.0x2.0mm, F.Cu at (240.7, 125.7)
- added TP5: TestPoint, TestPoint:TestPoint_Pad_2.0x2.0mm, F.Cu at (216.5, 55.9)
- added TP6: TestPoint, TestPoint:TestPoint_Pad_2.0x2.0mm, F.Cu at (212.1, 64.1)
- added TP7: TestPoint, TestPoint:TestPoint_Pad_2.0x2.0mm, F.Cu at (229.9, 47.6)
- added TP8: TestPoint, TestPoint:TestPoint_Pad_2.0x2.0mm, F.Cu at (236.2, 53.3)
- added TP9: TestPoint, TestPoint:TestPoint_Pad_2.0x2.0mm, F.Cu at (223.5, 47.6)
- added U10: ADA4891, Package_TO_SOT_SMD:TSOT-23-5, F.Cu at (199.3, 133.0)
- added U11: MIC5219-adj, Package_TO_SOT_SMD:SOT-23-5, F.Cu at (212.3, 123.8)
- added U12: ADC1175-50, Package_SO:TSSOP-24_4.4x7.8mm_P0.65mm, F.Cu at (229.2, 135.9)
- added U5: MIC5219-adj, Package_TO_SOT_SMD:SOT-23-5, F.Cu at (212.3, 75.6)
- added U6: ADC1175-50, Package_SO:TSSOP-24_4.4x7.8mm_P0.65mm, F.Cu at (229.2, 87.6)
- added U7: ADA4891, Package_TO_SOT_SMD:TSOT-23-5, F.Cu at (199.3, 108.9)
- added U8: MIC5219-adj, Package_TO_SOT_SMD:SOT-23-5, F.Cu at (212.3, 99.7)
- added U9: ADC1175-50, Package_SO:TSSOP-24_4.4x7.8mm_P0.65mm, F.Cu at (229.2, 111.8)
- C1: value 47p -> n.p.; footprint Capacitor_SMD:C_0805_2012Metric -> Capacitor_SMD:C_1206_3216Metric
- C10: value 100n -> 1u
- C11: value 62p -> 10u
- C13, C4: value 10u -> 100n; footprint Capacitor_SMD:C_1206_3216Metric -> Capacitor_SMD:C_0805_2012Metric
- C14, C5: footprint Capacitor_SMD:C_1206_3216Metric -> Capacitor_SMD:C_0805_2012Metric
- C16: value 10u -> n.p.
- C18: value 10u -> 2p, TBD; footprint Capacitor_SMD:C_1206_3216Metric -> Capacitor_SMD:C_0805_2012Metric
- C2: value 15p -> 100n
- C3: value 100n -> 2p, TBD
- C6: value 100n -> 47p
- C7: value 100n -> 470p
- C8, C9: value 10u -> 1u; footprint Capacitor_SMD:C_1206_3216Metric -> Capacitor_SMD:C_0805_2012Metric
- D1: value LM4040DBZ-4.1 -> SM4T15AY; footprint Package_TO_SOT_SMD:SOT-23 -> Diode_SMD:D_SMA_Handsoldering
- J1: value conn -> +5V Isense; footprint Connector_PinHeader_2.54mm:PinHeader_2x09_P2.54mm_Vertical -> Connector_PinHeader_2.54mm:PinHeader_1x02_P2.54mm_Vertical
- J2: value analog in -> +3.3V Isense
- R1: value 470 -> 0
- R10: value 110 -> 0
- R11: value 33 -> 0
- R12: value 33 -> 10k
- R19: value 10k -> 33
- R2: value 9M -> 0
- R3: value 1M -> 150k; footprint Resistor_SMD:R_0805_2012Metric -> Resistor_SMD:R_1206_3216Metric
- R4: value 10k -> 20
- R5: value 1k -> 0
- R6: value 100 -> 0
- R7: value 237 -> 4k5
- R8: value 150 -> 10k
- R9: value 237 -> 0
- RV1: value 5k -> 50k; footprint Resistor_SMD:R_0805_2012Metric -> Potentiometer_SMD:Potentiometer_Bourns_3269P_Horizontal
- RV2: value 500 -> 50k; footprint Resistor_SMD:R_0805_2012Metric -> Potentiometer_SMD:Potentiometer_Bourns_3269P_Horizontal
- U1: value ADA4622-1 -> ADA4891; footprint Package_TO_SOT_SMD:SOT-23-5 -> Package_TO_SOT_SMD:TSOT-23-5
- U2: value LMH6702 -> MIC5219-adj
- U3: value LMH6702 -> ADC1175-50; footprint Package_TO_SOT_SMD:SOT-23-5 -> Package_SO:TSSOP-24_4.4x7.8mm_P0.65mm
- U4: value ADC1175 -> ADA4891; footprint Package_SO:TSSOP-24_4.4x7.8mm_P0.65mm -> Package_TO_SOT_SMD:TSOT-23-5
- moved J1 131.7 mm to (255.3, 102.9), turned to 90 degrees
- moved J2 131.4 mm to (255.3, 82.5), turned to 90 degrees
- moved R2 125.8 mm to (251.5, 82.9), turned to 90 degrees
- moved C15 108.2 mm to (228.0, 56.2), turned to 270 degrees
- moved U3 108.1 mm to (229.2, 63.5), turned to 180 degrees
- moved R7 106.2 mm to (218.4, 51.8), turned to 90 degrees
- moved R1 105.1 mm to (255.6, 105.4), turned to 180 degrees
- moved R18 104.9 mm to (240.7, 61.6)
- moved C13 104.7 mm to (233.0, 55.5), turned to 90 degrees
- moved R16 104.2 mm to (240.7, 64.1)
- moved R15 103.9 mm to (236.9, 65.4)
- moved R14 103.6 mm to (240.7, 66.7)
- moved R13 103.3 mm to (236.9, 67.9)
- moved C7 102.7 mm to (212.1, 55.2), turned to 180 degrees
- moved R12 99.9 mm to (230.8, 52.1)
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Connections:
- C1 pad 2: GND -> Net-(C1-Pad2)
- C10 pad 1: -5V -> Net-(C10-Pad1)
- C12 pad 1: +5V -> Net-(C11-Pad1)
- C13 pad 1: -5V -> +3V3
- C14 pad 1: Net-(C14-Pad1) -> GND
- C14 pad 2: GND -> Net-(C14-Pad2)
- C15 pad 1: Net-(C14-Pad1) -> GND
- C15 pad 2: GND -> Net-(C14-Pad2)
- C16 pad 1: +5V -> Net-(C16-Pad1)
- C16 pad 2: GND -> Net-(C16-Pad2)
- C17 pad 1: -5V -> Net-(C17-Pad1)
- C18 pad 1: GND -> Net-(C18-Pad1)
- C18 pad 2: Net-(C18-Pad2) -> Net-(C16-Pad1)
- C19 pad 1: GND -> +5V
- C19 pad 2: Net-(C18-Pad2) -> GND
- C2 pad 1: Net-(C1-Pad1) -> Net-(C2-Pad1)
- C2 pad 2: analog-in -> GND
- C3 pad 1: +5V -> Net-(C3-Pad1)
- C3 pad 2: GND -> Net-(C1-Pad1)
- C4 pad 1: -5V -> +5V
- C6 pad 1: -5V -> Net-(C6-Pad1)
- C7 pad 1: +5V -> Net-(C7-Pad1)
- C8 pad 1: -5V -> Net-(C8-Pad1)
- C9 pad 1: +5V -> Net-(C9-Pad1)
- D1 pad 1: GND -> Net-(D1-Pad1)
- D1 pad 2: Net-(D1-Pad2) -> Net-(C1-Pad2)
- J1 pad 1: Net-(J1-Pad1) -> +5V
- J2 pad 1: GND -> Net-(J2-Pad1)
- J2 pad 2: analog-in -> +3V3
- L1 pad 1: Net-(C14-Pad1) -> Net-(C11-Pad1)
- L2 pad 1: Net-(C18-Pad2) -> Net-(C14-Pad2)
- L2 pad 2: Net-(C14-Pad1) -> Net-(C11-Pad1)
- R1 pad 1: +5V -> Net-(J1-Pad2)
- R1 pad 2: Net-(D1-Pad2) -> +5V
- R10 pad 1: Net-(C11-Pad1) -> Net-(C8-Pad1)
- R11 pad 1: Net-(R11-Pad1) -> Net-(C9-Pad1)
- R11 pad 2: Net-(J1-Pad1) -> Net-(R11-Pad2)
- R12 pad 1: Net-(R12-Pad1) -> Net-(J5-Pad2)
- R12 pad 2: Net-(J1-Pad2) -> GND
- R13 pad 2: Net-(J1-Pad3) -> /ADC1-D0
- R14 pad 2: Net-(J1-Pad4) -> /ADC1-D1
- R15 pad 2: Net-(J1-Pad5) -> /ADC1-D2
- R16 pad 2: Net-(J1-Pad6) -> /ADC1-D3
- R17 pad 2: Net-(J1-Pad7) -> /ADC1-D4
- R18 pad 2: Net-(J1-Pad8) -> /ADC1-D5
- R19 pad 1: VDD -> Net-(R19-Pad1)
- R19 pad 2: Net-(J1-Pad10) -> /ADC1-D6
- R2 pad 1: Net-(C1-Pad1) -> +3V3
- R2 pad 2: analog-in -> Net-(J2-Pad1)
- R3 pad 1: Net-(C1-Pad1) -> Net-(C1-Pad2)
- R3 pad 2: GND -> Net-(C1-Pad1)
- R4 pad 1: Net-(D1-Pad2) -> Net-(C6-Pad1)
- R4 pad 2: Net-(R4-Pad2) -> Net-(C3-Pad1)
- R5 pad 1: Net-(R4-Pad2) -> Net-(C8-Pad1)
- R5 pad 2: (no net) -> +5V
- R6 pad 1: Net-(R6-Pad1) -> Net-(C10-Pad1)
- R6 pad 2: (no net) -> Net-(C8-Pad1)
- R7 pad 1: Net-(R7-Pad1) -> Net-(C7-Pad1)
- R7 pad 2: Net-(R7-Pad2) -> Net-(C10-Pad1)
- R8 pad 2: Net-(R7-Pad1) -> Net-(C7-Pad1)
- R9 pad 1: Net-(R10-Pad2) -> GND
- R9 pad 2: Net-(R6-Pad1) -> Net-(C9-Pad1)
- RV1 pad 1: Net-(RV1-Pad1) -> Net-(C10-Pad1)
- RV1 pad 2: Net-(RV1-Pad1) -> Net-(C2-Pad1)
- RV2 pad 1: Net-(RV1-Pad1) -> Net-(C3-Pad1)
- RV2 pad 2: Net-(RV1-Pad1) -> Net-(C3-Pad1)
- U1 pad 1: Net-(R7-Pad2) -> Net-(C3-Pad1)
- U1 pad 2: +5V -> GND
- U1 pad 3: Net-(C1-Pad1) -> Net-(C2-Pad1)
- U1 pad 4: Net-(R7-Pad2) -> Net-(C1-Pad1)
- U1 pad 5: -5V -> +5V
- U2 pad 1: Net-(RV1-Pad1) -> +5V
- U2 pad 2: -5V -> GND
- U2 pad 3: GND -> +5V
- U2 pad 4: Net-(R4-Pad2) -> Net-(C7-Pad1)
- U2 pad 5: +5V -> Net-(C10-Pad1)
- U3 pad 1: Net-(R10-Pad2) -> Net-(J5-Pad2)
- U3 pad 2: -5V -> GND
- U3 pad 3: Net-(R7-Pad1) -> Net-(R13-Pad1)
- U3 pad 4: Net-(R6-Pad1) -> Net-(R14-Pad1)
- U3 pad 5: +5V -> Net-(R15-Pad1)
- U4 pad 1: Net-(J1-Pad10) -> Net-(C18-Pad1)
- U4 pad 3: Net-(R11-Pad1) -> Net-(C17-Pad1)
- U4 pad 4: Net-(R12-Pad1) -> Net-(C16-Pad1)
- U4 pad 5: Net-(R13-Pad1) -> +5V
Routing:
- net GND: track 0.00 -> 822.9 mm, vias 0 -> 68
- net +5V: track 0.00 -> 476.5 mm, vias 0 -> 21
- net +3V3: track 0.00 -> 158.1 mm, vias 0 -> 4
- net /ADC1-CLK: track 0.00 -> 37.9 mm
- net /ADC3-D0: track 0.00 -> 37.8 mm
- net /ADC3-D1: track 0.00 -> 37.1 mm
- net /ADC3-D2: track 0.00 -> 37.1 mm
- net /ADC3-CLK: track 0.00 -> 36.5 mm
- net /ADC3-D4: track 0.00 -> 36.5 mm
- net /ADC3-D6: track 0.00 -> 36.3 mm
- net /ADC3-D3: track 0.00 -> 35.8 mm
- net /ADC3-D5: track 0.00 -> 35.6 mm
- net /ADC3-D7: track 0.00 -> 35.6 mm
- net /ADC4-CLK: track 0.00 -> 34.6 mm
- net /ADC4-D2: track 0.00 -> 33.9 mm
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Other:
- board outline added: 98.4 x 99.1 mm
- net class Default: clearance 0.2 -> 0.2032; trace_width 0.25 -> 0.3048; via_dia 0.6 -> 1.016; via_drill 0.4 -> 0.508
- rule trace_clearance: 0.2 -> 0.2032
- rule trace_min: 0.2 -> 0.2032
- rule via_min_drill: 0.3 -> 0.508
- rule via_min_size: 0.4 -> 0.508

Commit message: first version, ordered at JLCPCB
Parts:
- added REF**: MountingHole_2.2mm_M2_Pad, MountingHole:MountingHole_2.2mm_M2_Pad, F.Cu at (254.0, 48.3)
- added REF**: MountingHole_2.2mm_M2_Pad, MountingHole:MountingHole_2.2mm_M2_Pad, F.Cu at (172.7, 48.3)
- added REF**: MountingHole_2.2mm_M2_Pad, MountingHole:MountingHole_2.2mm_M2_Pad, F.Cu at (172.7, 137.2)
- added REF**: MountingHole_2.2mm_M2_Pad, MountingHole:MountingHole_2.2mm_M2_Pad, F.Cu at (254.0, 137.2)
- added REF**: OSHW-Logo_11.4x12mm_SilkScreen, Symbol:OSHW-Logo_11.4x12mm_SilkScreen, F.Cu at (252.1, 59.1)
Routing:
- net +5V: track 476.5 -> 463.0 mm, vias 21 -> 26
- net /ADC1-CLK: track 37.9 -> 36.7 mm
- added copper zone on F.Cu, net +5V
- added copper zone on B.Cu, net GND
Other:
- board size 98.4 x 99.1 mm -> 99.7 x 99.1 mm
- board text added: "ADC4 Frank Buss REV 1"
- board text added: "in 1"
- board text added: "in 2"
- board text added: "in 3"
- board text added: "in 4"

Commit message: DDR3 RAM sample storage implemented
Parts:
- C18, C3, C33, C48: value 2p, TBD -> 0.5p
- R10, R11, R24, R29, R30, R43, R48, R49, R5, R62, R67, R68: value 0 -> n.p.
- R23, R4, R42, R61: value 20 -> 33
Changed lines of the file:
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@@
       (effects (font (size 1 1) (thickness 0.15)))
     )
-    (fp_text value 20 (at 0 1.65 180) (layer F.Fab)
+    (fp_text value 33 (at 0 1.65 180) (layer F.Fab)
       (effects (font (size 1 1) (thickness 0.15)))
     )
@@
       (effects (font (size 1 1) (thickness 0.15)))
     )
-    (fp_text value 0 (at 0 1.65) (layer F.Fab)
+    (fp_text value n.p. (at 0 1.65) (layer F.Fab)
       (effects (font (size 1 1) (thickness 0.15)))
     )
@@
       (effects (font (size 1 1) (thickness 0.15)))
     )
-    (fp_text value 0 (at 0 1.65 90) (layer F.Fab)
+    (fp_text value n.p. (at 0 1.65 90) (layer F.Fab)
       (effects (font (size 1 1) (thickness 0.15)))
     )
@@
       (effects (font (size 1 1) (thickness 0.15)))
     )
-    (fp_text value "2p, TBD" (at 0 1.65 180) (layer F.Fab)
+    (fp_text value 0.5p (at 0 1.65 180) (layer F.Fab)
       (effects (font (size 1 1) (thickness 0.15)))
     )
@@
       (effects (font (size 1 1) (thickness 0.15)))
     )
-    (fp_text value "2p, TBD" (at 0 1.65 180) (layer F.Fab)
+    (fp_text value 0.5p (at 0 1.65 180) (layer F.Fab)
       (effects (font (size 1 1) (thickness 0.15)))
     )
@@
       (effects (font (size 1 1) (thickness 0.15)))
     )
-    (fp_text value "2p, TBD" (at 0 1.65 180) (layer F.Fab)
+    (fp_text value 0.5p (at 0 1.65 180) (layer F.Fab)
       (effects (font (size 1 1) (thickness 0.15)))
     )
@@
       (effects (font (size 1 1) (thickness 0.15)))
     )
-    (fp_text value "2p, TBD" (at 0 1.65 180) (layer F.Fab)
+    (fp_text value 0.5p (at 0 1.65 180) (layer F.Fab)
       (effects (font (size 1 1) (thickness 0.15)))
     )
@@
       (effects (font (size 1 1) (thickness 0.15)))
     )
-    (fp_text value 0 (at 0 1.65) (layer F.Fab)
+    (fp_text value n.p. (at 0 1.65) (layer F.Fab)
       (effects (font (size 1 1) (thickness 0.15)))
     )
@@
       (effects (font (size 1 1) (thickness 0.15)))
     )
-    (fp_text value 20 (at 0 1.65 180) (layer F.Fab)
+    (fp_text value 33 (at 0 1.65 180) (layer F.Fab)
       (effects (font (size 1 1) (thickness 0.15)))
     )
@@
       (effects (font (size 1 1) (thickness 0.15)))
     )
-    (fp_text value 0 (at 0 1.65 90) (layer F.Fab)
+    (fp_text value n.p. (at 0 1.65 90) (layer F.Fab)
       (effects (font (size 1 1) (thickness 0.15)))
     )
@@
       (effects (font (size 1 1) (thickness 0.15)))
     )
-    (fp_text value 0 (at 0 1.65) (layer F.Fab)
+    (fp_text value n.p. (at 0 1.65) (layer F.Fab)
       (effects (font (size 1 1) (thickness 0.15)))
     )
@@
       (effects (font (size 1 1) (thickness 0.15)))
     )
-    (fp_text value 0 (at 0 1.65) (layer F.Fab)
+    (fp_text value n.p. (at 0 1.65) (layer F.Fab)
       (effects (font (size 1 1) (thickness 0.15)))
     )
@@
       (effects (font (size 1 1) (thickness 0.15)))
     )
-    (fp_text value 20 (at 0 1.65 180) (layer F.Fab)
+    (fp_text value 33 (at 0 1.65 180) (layer F.Fab)
       (effects (font (size 1 1) (thickness 0.15)))
     )
@@
       (effects (font (size 1 1) (thickness 0.15)))
     )
-    (fp_text value 0 (at 0 1.65 90) (layer F.Fab)
+    (fp_text value n.p. (at 0 1.65 90) (layer F.Fab)
       (effects (font (size 1 1) (thickness 0.15)))
     )
@@
       (effects (font (size 1 1) (thickness 0.15)))
     )
-    (fp_text value 0 (at 0 1.65) (layer F.Fab)
+    (fp_text value n.p. (at 0 1.65) (layer F.Fab)
       (effects (font (size 1 1) (thickness 0.15)))
     )
@@
       (effects (font (size 1 1) (thickness 0.15)))
     )
-    (fp_text value 0 (at 0 1.65) (layer F.Fab)
+    (fp_text value n.p. (at 0 1.65) (layer F.Fab)
       (effects (font (size 1 1) (thickness 0.15)))
     )
@@
       (effects (font (size 1 1) (thickness 0.15)))
     )
-    (fp_text value 20 (at 0 1.65 180) (layer F.Fab)
+    (fp_text value 33 (at 0 1.65 180) (layer F.Fab)
       (effects (font (size 1 1) (thickness 0.15)))
     )
@@
       (effects (font (size 1 1) (thickness 0.15)))
     )
-    (fp_text value 0 (at 0 1.65 90) (layer F.Fab)
+    (fp_text value n.p. (at 0 1.65 90) (layer F.Fab)
       (effects (font (size 1 1) (thickness 0.15)))
     )
@@
       (effects (font (size 1 1) (thickness 0.15)))
     )
-    (fp_text value 0 (at 0 1.65) (layer F.Fab)
+    (fp_text value n.p. (at 0 1.65) (layer F.Fab)
       (effects (font (size 1 1) (thickness 0.15)))
     )
@@
       (effects (font (size 1 1) (thickness 0.15)))
     )
-    (fp_text value 0 (at 0 1.65) (layer F.Fab)
+    (fp_text value n.p. (at 0 1.65) (layer F.Fab)
       (effects (font (size 1 1) (thickness 0.15)))
     )
